File: PiDGC PCB/PiDGC.brd (EAGLE design)
At the start: 57.1 x 58.1 mm, 26 parts, among them IC1 3.3V

Commit message: More work
Connections:
- net N$10 renamed ANALOG1_IN
- net N$2 renamed IGNITION
- net N$3 renamed HIGHBEAM_IN
- net N$35 renamed IGNITION_IN
- net N$36 renamed VSS_IN
- net N$6 renamed LOWBEAM_IN
- net N$7 renamed REVERSE_IN
- net N$8 renamed RIGHTSIG_IN
- net N$9 renamed LEFTSIG_IN
Changed lines of the file:
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@@
 <wire x1="2.54" y1="45.72" x2="2.54" y2="38.1" width="0.3048" layer="16"/>
 </signal>
-<signal name="N$6">
+<signal name="LOWBEAM_IN">
 <contactref element="U$1" pad="10/CS"/>
 <contactref element="R1" pad="13"/>
@@
 <via x="39.0144" y="49.0728" extent="1-16" drill="0.35"/>
 </signal>
-<signal name="N$7">
+<signal name="REVERSE_IN">
 <contactref element="U$1" pad="9/CS"/>
 <contactref element="R1" pad="12"/>
@@
 <wire x1="46.9392" y1="51.3588" x2="46.93" y2="51.435" width="0.1524" layer="1"/>
 </signal>
-<signal name="N$8">
+<signal name="RIGHTSIG_IN">
 <contactref element="U$1" pad="8"/>
 <contactref element="R1" pad="11"/>
@@
 <via x="49.6824" y="50.5968" extent="1-16" drill="0.35"/>
 </signal>
-<signal name="N$9">
+<signal name="LEFTSIG_IN">
 <contactref element="U$1" pad="7"/>
 <contactref element="R1" pad="10"/>
@@
 <via x="50.292" y="49.8348" extent="1-16" drill="0.35"/>
 </signal>
-<signal name="N$10">
+<signal name="ANALOG1_IN">
 <contactref element="U$1" pad="15/A1"/>
 <contactref element="R1" pad="9"/>
@@
 <wire x1="6.35" y1="19.05" x2="6.35" y2="34.29" width="0.3048" layer="16"/>
 </signal>
-<signal name="N$35">
+<signal name="IGNITION_IN">
 <contactref element="U$1" pad="14/A0"/>
 <contactref element="R1" pad="16"/>
@@
 <wire x1="40.6908" y1="46.3296" x2="40.7" y2="46.355" width="0.1524" layer="1"/>
 </signal>
-<signal name="N$3">
+<signal name="HIGHBEAM_IN">
 <contactref element="U$1" pad="11/MOSI"/>
 <contactref element="R1" pad="14"/>
@@
 <via x="26.5176" y="37.1856" extent="1-16" drill="0.35"/>
 </signal>
-<signal name="N$36">
+<signal name="VSS_IN">
 <contactref element="U$1" pad="12/MISO"/>
 <contactref element="R1" pad="15"/>
@@
 <via x="48.6156" y="46.482" extent="1-16" drill="0.35"/>
 </signal>
-<signal name="N$2">
+<signal name="IGNITION">
 <contactref element="IC1" pad="3"/>
 <contactref element="C1" pad="+"/>
