File: PiDGC PCB/PiDGC.sch (EAGLE design)
At the start: 26 parts, among them IC1 3.3V

Commit message: More work
Connections:
- net N$10 renamed ANALOG1_IN
- net N$2 renamed IGNITION
- net N$3 renamed HIGHBEAM_IN
- net N$35 renamed IGNITION_IN
- net N$36 renamed VSS_IN
- net N$6 renamed LOWBEAM_IN
- net N$7 renamed REVERSE_IN
- net N$8 renamed RIGHTSIG_IN
- net N$9 renamed LEFTSIG_IN
Changed lines of the file:
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@@
 </instance>
 <instance part="FUELSENSOR" gate="G$1" x="55.88" y="71.12" smashed="yes" rot="R180">
-<attribute name="NAME" x="73.025" y="72.0598" size="1.778" layer="95" rot="R180"/>
+<attribute name="NAME" x="73.787" y="73.3298" size="1.778" layer="95" rot="R180"/>
 <attribute name="VALUE" x="57.023" y="74.422" size="1.778" layer="96" rot="R180"/>
 </instance>
@@
 </segment>
 </net>
-<net name="N$6" class="0">
+<net name="LOWBEAM_IN" class="0">
 <segment>
 <wire x1="38.1" y1="-22.86" x2="25.4" y2="-22.86" width="0.1524" layer="91"/>
@@
 <pinref part="R1" gate="B" pin="13"/>
 <pinref part="R3" gate="B" pin="4"/>
-</segment>
-</net>
-<net name="N$7" class="0">
+<label x="25.4" y="-12.7" size="1.778" layer="95" rot="R90"/>
+</segment>
+</net>
+<net name="REVERSE_IN" class="0">
 <segment>
 <wire x1="7.62" y1="-25.4" x2="22.86" y2="-25.4" width="0.1524" layer="91"/>
@@
 <pinref part="R1" gate="B" pin="12"/>
 <pinref part="R3" gate="B" pin="5"/>
-</segment>
-</net>
-<net name="N$8" class="0">
+<label x="22.86" y="-12.7" size="1.778" layer="95" rot="R90"/>
+</segment>
+</net>
+<net name="RIGHTSIG_IN" class="0">
 <segment>
 <wire x1="38.1" y1="-27.94" x2="20.32" y2="-27.94" width="0.1524" layer="91"/>
@@
 <pinref part="R1" gate="B" pin="11"/>
 <pinref part="R3" gate="B" pin="6"/>
-</segment>
-</net>
-<net name="N$9" class="0">
+<label x="20.32" y="-12.7" size="1.778" layer="95" rot="R90"/>
+</segment>
+</net>
+<net name="LEFTSIG_IN" class="0">
 <segment>
 <wire x1="7.62" y1="-30.48" x2="17.78" y2="-30.48" width="0.1524" layer="91"/>
@@
 <pinref part="R1" gate="B" pin="10"/>
 <pinref part="R3" gate="B" pin="7"/>
-</segment>
-</net>
-<net name="N$10" class="0">
+<label x="17.78" y="-12.7" size="1.778" layer="95" rot="R90"/>
+</segment>
+</net>
+<net name="ANALOG1_IN" class="0">
 <segment>
 <wire x1="38.1" y1="-33.02" x2="35.56" y2="-33.02" width="0.1524" layer="91"/>
@@
 <pinref part="R1" gate="B" pin="9"/>
 <pinref part="R3" gate="B" pin="8"/>
+<label x="35.56" y="-12.7" size="1.778" layer="95" rot="R90"/>
 </segment>
 </net>
@@
 </segment>
 </net>
-<net name="N$35" class="0">
+<net name="IGNITION_IN" class="0">
 <segment>
 <wire x1="7.62" y1="-15.24" x2="33.02" y2="-15.24" width="0.1524" layer="91"/>
@@
 <pinref part="R1" gate="B" pin="16"/>
 <pinref part="R3" gate="B" pin="1"/>
-</segment>
-</net>
-<net name="N$3" class="0">
+<label x="33.02" y="-12.7" size="1.778" layer="95" rot="R90"/>
+</segment>
+</net>
+<net name="HIGHBEAM_IN" class="0">
 <segment>
 <wire x1="7.62" y1="-20.32" x2="27.94" y2="-20.32" width="0.1524" layer="91"/>
@@
 <pinref part="R1" gate="B" pin="14"/>
 <pinref part="R3" gate="B" pin="3"/>
-</segment>
-</net>
-<net name="N$36" class="0">
+<label x="27.94" y="-12.7" size="1.778" layer="95" rot="R90"/>
+</segment>
+</net>
+<net name="VSS_IN" class="0">
 <segment>
 <wire x1="38.1" y1="-17.78" x2="30.48" y2="-17.78" width="0.1524" layer="91"/>
@@
 <pinref part="R1" gate="B" pin="15"/>
 <pinref part="R3" gate="B" pin="2"/>
-</segment>
-</net>
-<net name="N$2" class="0">
+<label x="30.48" y="-12.7" size="1.778" layer="95" rot="R90"/>
+</segment>
+</net>
+<net name="IGNITION" class="0">
 <segment>
 <pinref part="IC1" gate="A1" pin="VI"/>
@@
 <junction x="101.6" y="93.98"/>
 <pinref part="R3" gate="B" pin="16"/>
-</segment>
-</net>
+<label x="54.356" y="-14.732" size="1.778" layer="95"/>
+</segment>
+</net>
